File: Alexandrie.kicad_pcb (KiCad board)
At the start: 2 copper layers, 100 x 100 mm, 56 parts, among them J1 Conn_01x03, J10 Conn_01x07, J2 Conn_02x05_Odd_Even, J3 CONN_01X03, J4 Conn_01x06, J5 Conn_02x05_Odd_Even, J6 Conn_02x05_Odd_Even, J7 Conn_01x05, J8 Conn_02x05_Odd_Even, J9 Conn_01x04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

Commit message: first RTM with silkmask
Parts:
- C7, C8, R4, R6: moved to B.Cu
- moved C5 113.4 mm to (135.0, 130.5), turned to -90 degrees
- moved C4 102.8 mm to (136.5, 107.0), turned to 90 degrees
- moved C8 100.0 mm to (126.0, 117.0), turned to -90 degrees
- moved C6 91.1 mm to (137.5, 76.0), turned to -90 degrees
- moved C7 89.1 mm to (130.0, 90.0)
- moved C1 85.6 mm to (116.5, 97.0)
- moved C13 82.0 mm to (101.5, 124.0)
- moved C9 80.5 mm to (107.5, 111.0)
- moved C11 80.5 mm to (107.5, 114.0)
- moved R1 80.4 mm to (116.5, 100.5), turned to 180 degrees
- moved C2 78.5 mm to (118.0, 84.0)
- moved C3 74.7 mm to (122.0, 59.5), turned to 180 degrees
- moved R4 72.7 mm to (110.5, 104.5), turned to 180 degrees
- moved R2 71.7 mm to (111.0, 96.5), turned to 180 degrees
- moved R3 69.1 mm to (116.0, 88.5), turned to -90 degrees
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Routing:
- net +5V: track 248.9 -> 300.5 mm, vias 19 -> 21
- net GND: track 113.0 -> 129.8 mm, vias 73 -> 229
- net Net-(J4-Pin_6): track 34.5 -> 46.6 mm
- net SPI_SPL_CLK: track 29.6 -> 39.5 mm
- net SPI_SPL_Data: track 40.7 -> 46.9 mm
- net +12V: track 234.4 -> 237.5 mm
- net SPI_TX_Load: track 28.8 -> 31.5 mm
- net SPI_RX_Load: track 41.9 -> 44.5 mm
- net Net-(D2-A): track 2.01 -> 3.21 mm
Other:
- board text added: "+12V 6m_Bypass 17/15m 40m 160m"
- board text added: "12V NC 15M 9.5M 20M"
- board text added: "12V RX2_GND 15MHz 9.5MHz 20MHz"
- board text added: "Ext.PWR"
- board text added: "GND Ant_Tune SPI_TX_Load SPI_CLK +12V Alex"
- board text added: "GND Att2 Att1 TX_RX_RLY"
- board text added: "GND By-Pass 6m_LNA 6.5_MHz 13_MHz"
- board text added: "GND GND 12/10m 30/20m 80m"
- board text added: "J16 PWR"
- board text added: "REFL FWD RX_Load Data GND"
- board text removed: "Ant_Tune +12V Alex SPI_SDO SPI_SCK SPI_RX_Load SPI_TX_Load FWD_PWR PTT REFL_PWR GND"
- board text removed: "Ext."
- board text removed: "FWD_PWR REFL_PWR Gnd +12V TX_RX_RLY"
- board text removed: "Gnd +12V HPF_ByPass Gnd 6mLNA 1.5HPF 6.5HPF 9.5HPF 13HPF 20HPF Att2 Att1 TX_RX_RLY"
- board text removed: "Gnd +12V TX_RX_RLY 6m 12/10m 17/15m 6m 30/20m 40m 80m 160m"
- board text removed: "J16"
- board text removed: "PWR"

Commit message: DRC clean, iBom saved
Parts:
- moved C12 11.4 mm to (119.5, 114.5), turned to 90 degrees
- moved U10 4.38 mm to (114.0, 122.3), turned to -90 degrees
- moved C13 3.54 mm to (102.0, 127.5)
- moved D1 0.50 mm to (106.0, 121.0)
Connections:
- U10 pad 1: +5V -> +12V
- U10 pad 3: +12V -> +5V
Routing:
- net +12V: track 237.5 -> 273.4 mm
- net SPI_SPL_Data: track 46.9 -> 45.9 mm
- net 6mLNA: track 41.1 -> 40.4 mm
- net 20HPF: track 35.3 -> 34.6 mm
- net Net-(D2-K): track 4.20 -> 3.53 mm
- net 13HPF: track 37.2 -> 36.6 mm
- net +5V: track 300.5 -> 299.9 mm
- net Net-(D1-A): track 4.28 -> 4.78 mm
- net GND: vias 229 -> 261

Commit message: minor chages, new iBom
Routing:
- net GND: vias 261 -> 294

Commit message: kicad 10 update, new readme, new wiki link
Parts:
- added J11: Conn_02x06_Odd_Even, Connector_IDC:IDC-Header_2x06_P2.54mm_Vertical, F.Cu at (176.0, 104.2)
- U1, U2: value 74HCT04 -> 74ACT04
Connections:
- J8 pad 8: GND -> TX_RX_RLY
Routing:
- net 9.5HPF: track 12.6 -> 71.8 mm, vias 0 -> 1
- net 6mLNA: track 40.4 -> 89.3 mm
- net 13HPF: track 36.6 -> 77.6 mm, vias 3 -> 4
- net 20HPF: track 34.6 -> 72.0 mm, vias 2 -> 3
- net +12V: track 273.4 -> 299.9 mm, vias 10 -> 12
- net 1.5HPF: track 17.9 -> 40.1 mm
- net Att2: track 29.2 -> 47.0 mm, vias 2 -> 4
- net 6.5HPF: track 26.5 -> 40.5 mm
- net Att1: track 28.3 -> 39.7 mm
- net HPF_ByPass: track 48.4 -> 57.4 mm
- net GND: track 129.8 -> 132.4 mm, vias 294 -> 297
Other:
- board text added: "Alex BPF-1"
- board text added: "Alex BPF-2"
- board text added: "Alex HPF-->"
- board text added: "Alex LPF"
- board text added: "Staight HPF flat cable"
- board text removed: "GND GND 12/10m 30/20m 80m"
- board text removed: "To Alex BPF-2"
- board text removed: "To Alex HPF/BPF-1"
- board text removed: "To Alex LPF"
